File: PCB/star_wars_arcade_sound_pcb/Sheet15A.kicad_sch (KiCad schematic)
At the start: 20 parts

Commit message: Began PCB layout
Parts:
- J_3: footprint (none) -> atari:DIP16
- J_5, K_5: footprint (none) -> atari:DIP20
- K_3: footprint (none) -> atari:DDIP40
Changed lines of the file:
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@@
       (effects (font (size 1.27 1.27)) (justify left))
     )
-    (property "Footprint" "" (id 2) (at 140.97 47.625 0)
+    (property "Footprint" "atari:DIP20" (id 2) (at 140.97 47.625 0)
       (effects (font (size 1.27 1.27)) hide)
     )
@@
       (effects (font (size 1.27 1.27)) (justify left))
     )
-    (property "Footprint" "" (id 2) (at 252.095 106.045 0)
+    (property "Footprint" "atari:DDIP40" (id 2) (at 252.095 106.045 0)
       (effects (font (size 1.27 1.27)) hide)
     )
@@
       (effects (font (size 1.27 1.27)) (justify left))
     )
-    (property "Footprint" "" (id 2) (at 142.24 131.445 0)
+    (property "Footprint" "atari:DIP20" (id 2) (at 142.24 131.445 0)
       (effects (font (size 1.27 1.27)) hide)
     )
@@
     (property "Reference" "J_3" (id 0) (at 48.895 95.885 0))
     (property "Value" "74LS139" (id 1) (at 48.895 99.06 0))
-    (property "Footprint" "" (id 2) (at 48.895 97.155 0)
-      (effects (font (size 1.27 1.27)) hide)
-    )
+    (property "Footprint" "atari:DIP16" (id 2) (at 48.895 97.155 0)
+      (effects (font (size 1.27 1.27)) hide)
+    )

Commit message: ICs placed
Parts:
- F/H_5, H_2, H_5: footprint (none) -> atari:DIP14
- F_5: footprint (none) -> atari:DIP16
Changed lines of the file:
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@@
       (effects (font (size 1.27 1.27)) (justify left))
     )
-    (property "Footprint" "" (id 2) (at 213.995 36.83 0)
+    (property "Footprint" "atari:DIP14" (id 2) (at 213.995 36.83 0)
       (effects (font (size 1.27 1.27)) hide)
     )
@@
     (property "Reference" "H_2" (id 0) (at 81.915 52.07 0))
     (property "Value" "74LS04" (id 1) (at 82.55 57.15 0))
-    (property "Footprint" "" (id 2) (at 78.105 54.61 0)
+    (property "Footprint" "atari:DIP14" (id 2) (at 78.105 54.61 0)
       (effects (font (size 1.27 1.27)) hide)
     )
@@
     (property "Reference" "F/H_5" (id 0) (at 250.19 131.445 0))
     (property "Value" "74LS125" (id 1) (at 250.19 126.365 0))
-    (property "Footprint" "" (id 2) (at 245.11 128.905 0)
+    (property "Footprint" "atari:DIP14" (id 2) (at 245.11 128.905 0)
       (effects (font (size 1.27 1.27)) hide)
     )
@@
       (effects (font (size 1.27 1.27)) (justify left))
     )
-    (property "Footprint" "" (id 2) (at 144.78 86.995 0)
+    (property "Footprint" "atari:DIP14" (id 2) (at 144.78 86.995 0)
       (effects (font (size 1.27 1.27)) hide)
     )
@@
       (effects (font (size 1.27 1.27)) (justify left))
     )
-    (property "Footprint" "" (id 2) (at 45.72 52.07 0)
+    (property "Footprint" "atari:DIP16" (id 2) (at 45.72 52.07 0)
       (effects (font (size 1.27 1.27)) hide)
     )
@@
     (property "Reference" "F/H_5" (id 0) (at 217.17 32.385 0))
     (property "Value" "74LS125" (id 1) (at 219.71 40.005 0))
-    (property "Footprint" "" (id 2) (at 214.63 37.465 0)
+    (property "Footprint" "atari:DIP14" (id 2) (at 214.63 37.465 0)
       (effects (font (size 1.27 1.27)) hide)
     )
@@
     (property "Reference" "F/H_5" (id 0) (at 250.825 150.495 0))
     (property "Value" "74LS125" (id 1) (at 250.19 146.05 0))
-    (property "Footprint" "" (id 2) (at 245.11 148.59 0)
+    (property "Footprint" "atari:DIP14" (id 2) (at 245.11 148.59 0)
       (effects (font (size 1.27 1.27)) hide)
     )
@@
       (effects (font (size 1.27 1.27)) (justify left))
     )
-    (property "Footprint" "" (id 2) (at 148.59 86.995 0)
+    (property "Footprint" "atari:DIP14" (id 2) (at 148.59 86.995 0)
       (effects (font (size 1.27 1.27)) hide)
     )
@@
       (effects (font (size 1.27 1.27)) (justify left))
     )
-    (property "Footprint" "" (id 2) (at 137.795 173.99 0)
-      (effects (font (size 1.27 1.27)) hide)
-    )
+    (property "Footprint" "atari:DIP14" (id 2) (at 137.795 173.99 0)
+      (effects (font (size 1.27 1.27)) hide)
+    )

Commit message: Placed all components
Parts:
- C1, C12, C6, C61, C8, C9, R1, R2, R3, R4: footprint (none) -> atari:GenericComp
- TP1, TP2: footprint (none) -> atari:TEST_POINT
Changed lines of the file:
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@@
       (effects (font (size 1.27 1.27)) (justify left))
     )
-    (property "Footprint" "" (id 2) (at 232.664 52.959 90)
+    (property "Footprint" "atari:GenericComp" (id 2) (at 232.664 52.959 90)
       (effects (font (size 1.27 1.27)) hide)
     )
@@
       (effects (font (size 1.27 1.27)) (justify left))
     )
-    (property "Footprint" "" (id 2) (at 23.241 26.924 90)
+    (property "Footprint" "atari:GenericComp" (id 2) (at 23.241 26.924 90)
       (effects (font (size 1.27 1.27)) hide)
     )
@@
       (effects (font (size 1.27 1.27)) (justify left))
     )
-    (property "Footprint" "" (id 2) (at 232.664 49.149 90)
+    (property "Footprint" "atari:GenericComp" (id 2) (at 232.664 49.149 90)
       (effects (font (size 1.27 1.27)) hide)
     )
@@
     (property "Reference" "C1" (id 0) (at 259.715 32.385 90))
     (property "Value" ".1uf" (id 1) (at 260.35 29.845 90))
-    (property "Footprint" "" (id 2) (at 260.985 30.1498 0)
+    (property "Footprint" "atari:GenericComp" (id 2) (at 260.985 30.1498 0)
       (effects (font (size 1.27 1.27)) hide)
     )
@@
     (property "Reference" "C61" (id 0) (at 207.645 28.575 90))
     (property "Value" ".1uf" (id 1) (at 208.28 26.035 90))
-    (property "Footprint" "" (id 2) (at 208.915 26.3398 0)
+    (property "Footprint" "atari:GenericComp" (id 2) (at 208.915 26.3398 0)
       (effects (font (size 1.27 1.27)) hide)
     )
@@
       (effects (font (size 1.27 1.27)) (justify left) hide)
     )
-    (property "Footprint" "" (id 2) (at 231.14 44.45 0)
+    (property "Footprint" "atari:TEST_POINT" (id 2) (at 231.14 44.45 0)
       (effects (font (size 1.27 1.27)) hide)
     )
@@
       (effects (font (size 1.27 1.27)) (justify left) hide)
     )
-    (property "Footprint" "" (id 2) (at 237.49 35.56 0)
+    (property "Footprint" "atari:TEST_POINT" (id 2) (at 237.49 35.56 0)
       (effects (font (size 1.27 1.27)) hide)
     )
@@
       (effects (font (size 1.27 1.27)) (justify left))
     )
-    (property "Footprint" "" (id 2) (at 232.156 32.639 90)
+    (property "Footprint" "atari:GenericComp" (id 2) (at 232.156 32.639 90)
       (effects (font (size 1.27 1.27)) hide)
     )
@@
     (property "Reference" "C8" (id 0) (at 149.225 27.94 90))
     (property "Value" ".1uf" (id 1) (at 149.86 25.4 90))
-    (property "Footprint" "" (id 2) (at 150.495 25.7048 0)
+    (property "Footprint" "atari:GenericComp" (id 2) (at 150.495 25.7048 0)
       (effects (font (size 1.27 1.27)) hide)
     )
@@
     (property "Reference" "C12" (id 0) (at 149.86 110.49 90))
     (property "Value" ".1uf" (id 1) (at 150.495 107.95 90))
-    (property "Footprint" "" (id 2) (at 151.13 108.2548 0)
+    (property "Footprint" "atari:GenericComp" (id 2) (at 151.13 108.2548 0)
       (effects (font (size 1.27 1.27)) hide)
     )
@@
     (property "Reference" "C6" (id 0) (at 59.69 41.91 90))
     (property "Value" ".1uf" (id 1) (at 60.325 39.37 90))
-    (property "Footprint" "" (id 2) (at 60.96 39.6748 0)
+    (property "Footprint" "atari:GenericComp" (id 2) (at 60.96 39.6748 0)
       (effects (font (size 1.27 1.27)) hide)
     )
@@
     (property "Reference" "C9" (id 0) (at 156.21 77.47 90))
     (property "Value" ".1uf" (id 1) (at 156.845 74.93 90))
-    (property "Footprint" "" (id 2) (at 157.48 75.2348 0)
-      (effects (font (size 1.27 1.27)) hide)
-    )
+    (property "Footprint" "atari:GenericComp" (id 2) (at 157.48 75.2348 0)
+      (effects (font (size 1.27 1.27)) hide)
+    )
