File: PCB/star_wars_arcade_sound_pcb/Sheet16A.kicad_sch (KiCad schematic)
At the start: 61 parts, among them Q1 2N3906, Q2 2N3906, Q3 2N3904

Commit message: Finished schematic
Changed lines of the file:
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@@
   (symbol (lib_id "atari:TL084") (at 127.635 187.325 0) (mirror x) (unit 3)
     (in_bom yes) (on_board yes)
-    (property "Reference" "C_4" (id 0) (at 132.715 189.23 0))
-    (property "Value" "TL084" (id 1) (at 134.62 184.15 0))
+    (property "Reference" "C_4" (id 0) (at 125.73 188.595 0))
+    (property "Value" "TL084" (id 1) (at 126.365 186.69 0))
     (property "Footprint" "" (id 2) (at 126.365 189.865 0)
       (effects (font (size 1.27 1.27)) hide)
@@
   (symbol (lib_id "atari:74LS04") (at 222.25 179.705 0) (unit 6)
     (in_bom yes) (on_board yes)
-    (property "Reference" "H_2" (id 0) (at 224.79 177.165 0))
+    (property "Reference" "H_2" (id 0) (at 220.98 179.705 0))
     (property "Value" "74LS04" (id 1) (at 226.695 182.245 0))
     (property "Footprint" "" (id 2) (at 222.25 179.705 0)
@@
       (effects (font (size 1.27 1.27)) (justify left))
     )
-    (property "Value" "TL084" (id 1) (at 44.45 184.785 0)
+    (property "Value" "TL084" (id 1) (at 45.085 184.785 0)
       (effects (font (size 1.27 1.27)) (justify left))
     )
@@
   (symbol (lib_id "atari:TL084") (at 41.91 215.265 0) (mirror x) (unit 2)
     (in_bom yes) (on_board yes)
-    (property "Reference" "C_3" (id 0) (at 46.99 217.17 0))
-    (property "Value" "TL084" (id 1) (at 48.895 212.09 0))
+    (property "Reference" "C_3" (id 0) (at 40.64 216.535 0))
+    (property "Value" "TL084" (id 1) (at 40.64 214.63 0))
     (property "Footprint" "" (id 2) (at 40.64 217.805 0)
       (effects (font (size 1.27 1.27)) hide)
@@
   (symbol (lib_id "atari:TL084") (at 47.625 234.95 0) (mirror x) (unit 4)
     (in_bom yes) (on_board yes)
-    (property "Reference" "C_4" (id 0) (at 52.705 236.855 0))
-    (property "Value" "TL084" (id 1) (at 54.61 231.775 0))
+    (property "Reference" "C_4" (id 0) (at 46.355 236.22 0))
+    (property "Value" "TL084" (id 1) (at 46.355 234.315 0))
     (property "Footprint" "" (id 2) (at 46.355 237.49 0)
       (effects (font (size 1.27 1.27)) hide)
@@
   (symbol (lib_id "atari:TL084") (at 41.91 162.56 0) (mirror x) (unit 2)
     (in_bom yes) (on_board yes)
-    (property "Reference" "C_4" (id 0) (at 46.99 164.465 0))
-    (property "Value" "TL084" (id 1) (at 48.895 159.385 0))
+    (property "Reference" "C_4" (id 0) (at 40.64 163.83 0))
+    (property "Value" "TL084" (id 1) (at 40.64 161.925 0))
     (property "Footprint" "" (id 2) (at 40.64 165.1 0)
       (effects (font (size 1.27 1.27)) hide)

Commit message: Began PCB layout
Parts:
- D_2, D_3, D_4, D_5: footprint (none) -> atari:DDIP40
- Q1, Q2, Q3: footprint Package_TO_SOT_THT:TO-92_Inline -> (none)
Changed lines of the file:
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@@
       (effects (font (size 1.27 1.27)) (justify left))
     )
-    (property "Footprint" "" (id 2) (at 158.75 64.77 0)
+    (property "Footprint" "atari:DDIP40" (id 2) (at 158.75 64.77 0)
       (effects (font (size 1.27 1.27)) hide)
     )
@@
       (effects (font (size 1.27 1.27)) (justify left))
     )
-    (property "Footprint" "" (id 2) (at 40.64 64.77 0)
+    (property "Footprint" "atari:DDIP40" (id 2) (at 40.64 64.77 0)
       (effects (font (size 1.27 1.27)) hide)
     )
@@
       (effects (font (size 1.27 1.27)) (justify left))
     )
-    (property "Footprint" "Package_TO_SOT_THT:TO-92_Inline" (id 2) (at 347.345 178.435 0)
+    (property "Footprint" "" (id 2) (at 347.345 178.435 0)
       (effects (font (size 1.27 1.27) italic) (justify left) hide)
     )
@@
       (effects (font (size 1.27 1.27)) (justify left))
     )
-    (property "Footprint" "" (id 2) (at 80.01 64.77 0)
+    (property "Footprint" "atari:DDIP40" (id 2) (at 80.01 64.77 0)
       (effects (font (size 1.27 1.27)) hide)
     )
@@
       (effects (font (size 1.27 1.27)) (justify left))
     )
-    (property "Footprint" "Package_TO_SOT_THT:TO-92_Inline" (id 2) (at 321.31 168.275 0)
+    (property "Footprint" "" (id 2) (at 321.31 168.275 0)
       (effects (font (size 1.27 1.27) italic) (justify left) hide)
     )
@@
       (effects (font (size 1.27 1.27)) (justify left))
     )
-    (property "Footprint" "Package_TO_SOT_THT:TO-92_Inline" (id 2) (at 240.665 172.72 0)
+    (property "Footprint" "" (id 2) (at 240.665 172.72 0)
       (effects (font (size 1.27 1.27) italic) (justify left) hide)
     )
@@
       (effects (font (size 1.27 1.27)) (justify left))
     )
-    (property "Footprint" "" (id 2) (at 119.38 64.77 0)
-      (effects (font (size 1.27 1.27)) hide)
-    )
+    (property "Footprint" "atari:DDIP40" (id 2) (at 119.38 64.77 0)
+      (effects (font (size 1.27 1.27)) hide)
+    )

Commit message: ICs placed
Parts:
- C/D_1: footprint (none) -> atari:DIP28
- C_3, C_4, F_2, H_2: footprint (none) -> atari:DIP14
- F_3: footprint (none) -> atari:DIP16
Changed lines of the file:
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@@
       (effects (font (size 1.27 1.27)) (justify left))
     )
-    (property "Footprint" "" (id 2) (at 190.5 174.625 0)
+    (property "Footprint" "atari:DIP16" (id 2) (at 190.5 174.625 0)
       (effects (font (size 1.27 1.27)) hide)
     )
@@
     (property "Reference" "C_4" (id 0) (at 125.73 188.595 0))
     (property "Value" "TL084" (id 1) (at 126.365 186.69 0))
-    (property "Footprint" "" (id 2) (at 126.365 189.865 0)
+    (property "Footprint" "atari:DIP14" (id 2) (at 126.365 189.865 0)
       (effects (font (size 1.27 1.27)) hide)
     )
@@
     (property "Reference" "C_4" (id 0) (at 46.99 139.7 0))
     (property "Value" "TL084" (id 1) (at 47.625 134.62 0))
-    (property "Footprint" "" (id 2) (at 40.64 140.335 0)
+    (property "Footprint" "atari:DIP14" (id 2) (at 40.64 140.335 0)
       (effects (font (size 1.27 1.27)) hide)
     )
@@
     (property "Reference" "H_2" (id 0) (at 220.98 179.705 0))
     (property "Value" "74LS04" (id 1) (at 226.695 182.245 0))
-    (property "Footprint" "" (id 2) (at 222.25 179.705 0)
+    (property "Footprint" "atari:DIP14" (id 2) (at 222.25 179.705 0)
       (effects (font (size 1.27 1.27)) hide)
     )
@@
       (effects (font (size 1.27 1.27)) (justify left))
     )
-    (property "Footprint" "" (id 2) (at 344.805 66.675 0)
+    (property "Footprint" "atari:DIP28" (id 2) (at 344.805 66.675 0)
       (effects (font (size 1.27 1.27)) hide)
     )
@@
       (effects (font (size 1.27 1.27)) (justify left))
     )
-    (property "Footprint" "" (id 2) (at 40.64 135.255 0)
+    (property "Footprint" "atari:DIP14" (id 2) (at 40.64 135.255 0)
       (effects (font (size 1.27 1.27)) hide)
     )
@@
       (effects (font (size 1.27 1.27)) (justify left))
     )
-    (property "Footprint" "" (id 2) (at 250.825 201.93 0)
+    (property "Footprint" "atari:DIP14" (id 2) (at 250.825 201.93 0)
       (effects (font (size 1.27 1.27)) hide)
     )
@@
       (effects (font (size 1.27 1.27)) (justify left))
     )
-    (property "Footprint" "" (id 2) (at 40.64 187.325 0)
+    (property "Footprint" "atari:DIP14" (id 2) (at 40.64 187.325 0)
       (effects (font (size 1.27 1.27)) hide)
     )
@@
     (property "Reference" "C_3" (id 0) (at 40.64 216.535 0))
     (property "Value" "TL084" (id 1) (at 40.64 214.63 0))
-    (property "Footprint" "" (id 2) (at 40.64 217.805 0)
+    (property "Footprint" "atari:DIP14" (id 2) (at 40.64 217.805 0)
       (effects (font (size 1.27 1.27)) hide)
     )
@@
     (property "Reference" "C_4" (id 0) (at 46.355 236.22 0))
     (property "Value" "TL084" (id 1) (at 46.355 234.315 0))
-    (property "Footprint" "" (id 2) (at 46.355 237.49 0)
+    (property "Footprint" "atari:DIP14" (id 2) (at 46.355 237.49 0)
       (effects (font (size 1.27 1.27)) hide)
     )
@@
     (property "Reference" "C_3" (id 0) (at 46.99 191.77 0))
     (property "Value" "TL084" (id 1) (at 47.625 186.69 0))
-    (property "Footprint" "" (id 2) (at 40.64 192.405 0)
+    (property "Footprint" "atari:DIP14" (id 2) (at 40.64 192.405 0)
       (effects (font (size 1.27 1.27)) hide)
     )
@@
     (property "Reference" "F_2" (id 0) (at 251.46 182.245 0))
     (property "Value" "C04" (id 1) (at 250.825 184.15 0))
-    (property "Footprint" "" (id 2) (at 252.73 182.88 0)
+    (property "Footprint" "atari:DIP14" (id 2) (at 252.73 182.88 0)
       (effects (font (size 1.27 1.27)) hide)
     )
@@
     (property "Reference" "F_2" (id 0) (at 251.46 201.295 0))
     (property "Value" "C04" (id 1) (at 250.825 203.2 0))
-    (property "Footprint" "" (id 2) (at 252.73 201.93 0)
+    (property "Footprint" "atari:DIP14" (id 2) (at 252.73 201.93 0)
       (effects (font (size 1.27 1.27)) hide)
     )
@@
     (property "Reference" "C_4" (id 0) (at 40.64 163.83 0))
     (property "Value" "TL084" (id 1) (at 40.64 161.925 0))
-    (property "Footprint" "" (id 2) (at 40.64 165.1 0)
-      (effects (font (size 1.27 1.27)) hide)
-    )
+    (property "Footprint" "atari:DIP14" (id 2) (at 40.64 165.1 0)
+      (effects (font (size 1.27 1.27)) hide)
+    )

Commit message: Placed all components
Parts:
- C16, C17, C18, C19, C22, C23, C24, C25, C26, C27, C28, C29, C30, C31, C32, C33, C34, C35, C36, C37, C38, C39, C40, C41, C42, R10, R11, R12, R13, R14, R15, R16, R17, R18, R19, R20, R21, R22, R23, R24, R25, R26, R27, R28, R29, R30, R8, R9: footprint (none) -> atari:GenericComp
- Q1, Q2, Q3: footprint (none) -> atari:GenericTrans

Commit message: 331 connections remain
Connections:
- net +5V: now also Q2.1 (E), R14.2
Changed lines of the file:
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@@
   (junction (at 29.845 160.02) (diameter 0) (color 0 0 0 0)
+  )
+  (junction (at 318.77 163.195) (diameter 0) (color 0 0 0 0)
   )
   (junction (at 187.96 159.385) (diameter 0) (color 0 0 0 0)
@@
     (pin "2")
   )
+  (symbol (lib_id "power:+5V") (at 318.77 163.195 0) (unit 1)
+    (in_bom yes) (on_board yes)
+    (property "Reference" "#PWR0257" (id 0) (at 318.77 167.005 0)
+      (effects (font (size 1.27 1.27)) hide)
+    )
+    (property "Value" "+5V" (id 1) (at 321.31 160.655 0))
+    (property "Footprint" "" (id 2) (at 318.77 163.195 0)
+      (effects (font (size 1.27 1.27)) hide)
+    )
+    (property "Datasheet" "" (id 3) (at 318.77 163.195 0)
+      (effects (font (size 1.27 1.27)) hide)
+    )
+    (pin "1")
+  )
   (symbol (lib_id "power:PWR_FLAG") (at 347.345 121.92 0) (unit 1)
