File: PCB/star_wars_arcade_sound_pcb/star_wars_arcade_sound_pcb.kicad_pcb (KiCad board)
At the start: 2 copper layers, 292.1 x 227.3 mm, 162 parts, among them P1 sw_main_connector, P2 sw_aud_connector, P3 sw_audio_edge_connector, Q1 2N3906, Q2 2N3906, Q3 2N3904, Q4 2N3904

Commit message: 189 connections remain
Parts:
- moved R12 0.63 mm to (213.4, 135.9)
Routing:
- net P: track 127.4 -> 344.2 mm
- net SR~{W}: track 40.3 -> 231.3 mm, vias 4 -> 6
- net SD7: track 250.9 -> 437.7 mm
- net SD6: track 275.6 -> 453.9 mm
- net ~{SOUND}: track 28.3 -> 205.8 mm
- net CLKQ: track 41.7 -> 207.2 mm, vias 1 -> 2
- net PHI_E: track 155.3 -> 317.0 mm
- net AB0: track 9.65 -> 170.0 mm, vias 1 -> 2
- net R~{W}B: track 9.65 -> 154.0 mm, vias 1 -> 2
- net MAINFLAG: track 34.2 -> 172.6 mm
- net SOUNDFLAG: track 17.6 -> 155.5 mm
- net SD5: track 333.8 -> 446.6 mm
- net ~{SOUNDRST}: track 29.5 -> 130.9 mm
- net 6MHZ: track 31.0 -> 123.2 mm, vias 3 -> 4
- net Net-(F/H_1-Pad20): track 0.00 -> 92.0 mm
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
Commit message: Ground plane and mounting holes remain
Parts:
- moved R48 2.54 mm to (108.0, 130.8)
- moved R49 2.54 mm to (108.0, 133.3)
- moved R19 0.63 mm to (148.6, 203.8)
- moved R38 0.63 mm to (52.7, 148.6)
- renumbered R49 to R48, R48 to R49
Connections:
- R52 pad 1: Net-(B_2-Pad1) -> AUD
- R53 pad 1: AUD -> Net-(B_2-Pad1)
Routing:
- net +5V: track 1917.4 -> 2110.6 mm, vias 12 -> 14
- net ~{SRES}: track 50.8 -> 224.3 mm, vias 2 -> 3
- net +12V: track 344.2 -> 510.6 mm
- net SPEECH: track 3.81 -> 168.7 mm
- net -5V: track 349.4 -> 502.7 mm, vias 1 -> 3
- net PA3: track 194.6 -> 268.9 mm, vias 2 -> 3
- net PHI_E: track 317.0 -> 388.9 mm
- net AUD: track 73.1 -> 141.1 mm
- net Net-(B_2-Pad1): track 8.26 -> 59.9 mm
- net SA0: track 286.0 -> 336.4 mm
- net CO1: track 0.00 -> 39.9 mm
- net RCK: track 24.3 -> 63.8 mm
- net ~{SOUNDWR}: track 63.2 -> 102.4 mm
- net SR~{W}: track 231.3 -> 268.9 mm
- net SA11: track 85.6 -> 122.1 mm
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