File: PCB/star_wars_arcade_sound_pcb/star_wars_arcade_sound_pcb.kicad_pcb (KiCad board)
At the start: 2 copper layers, 292.1 x 227.3 mm, 168 parts, among them P1 sw_main_connector, P2 sw_aud_connector, P3 sw_audio_edge_connector, Q1 2N3906, Q2 2N3906, Q3 2N3904, Q4 2N3904

Commit message: Bottom keep out areas remain
Routing:
- net GND: track 1044.2 -> 1363.7 mm

Commit message: Consolidated keep out areas
Routing:
- net GND: track 1363.7 -> 1556.4 mm

Commit message: Completed PCB
Routing:
- net GND: track 1556.4 -> 1597.8 mm
- net +5V: track 2221.0 -> 2226.1 mm
Other:
- board text added: "Designed By Nick Mikstas"
