File: PCB/star_wars_arcade_sound_pcb/star_wars_arcade_sound_pcb.kicad_sch (KiCad schematic)
At the start: 0 parts

Commit message: Updated schematic
Other:
- note added: "Arcade Audio PCB Schematics"
- note removed: "Arcade Audio PCB"
